File: swallowtailkb/swallowtail_split.kicad_pcb (KiCad board)
At the start: 2 copper layers, 147.8 x 149.5 mm, 50 parts

Commit message: added case conf
Routing:
- net P7: track 8.64 -> 189.6 mm
- net P8: track 0.00 -> 147.3 mm
- net P6: track 125.5 -> 205.9 mm
- net GND: track 82.4 -> 2.54 mm
- net P18: track 149.8 -> 225.1 mm, vias 1 -> 3
- net P9: track 75.8 -> 131.5 mm
- net pinky_home: track 0.00 -> 29.9 mm
- net ring_home: track 0.00 -> 28.9 mm
- net middle_top: track 0.00 -> 28.9 mm
- net ring_top: track 0.00 -> 28.9 mm
- net pinky_top: track 0.00 -> 28.9 mm
- net middle_bottom: track 0.00 -> 28.9 mm
- net ring_bottom: track 0.00 -> 28.9 mm
- net middle_home: track 0.00 -> 28.9 mm
- net P10: track 172.5 -> 148.3 mm
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- added copper zone on B.Cu, net GND
- added copper zone on F.Cu, net GND
Other:
- board text added: "Place MCU chip DOWN"
- board text added: "Place MCU chip UP"
